Commit message: somethings

File: my_robot_cell/my_robot_cell_description/urdf/my_robot_cell_macro.xacro (robot description, xacro)
@@ -34,5 +34,5 @@
       <visual>
         <geometry>
-          <mesh filename="package://my_robot_cell_description/meshes/ZenPoolWithToolBox.stl"/>
+          <mesh filename="package://my_robot_cell_description/meshes/environment/ZenPoolWithToolBox.stl"/>
         </geometry>
         <origin rpy="0 0 0" xyz="0.0 0.0 0.0"/>
@@ -41,5 +41,5 @@
       <collision>
         <geometry>
-          <mesh filename="package://my_robot_cell_description/meshes/ZenPoolWithToolBoxCollision.stl"/>
+          <mesh filename="package://my_robot_cell_description/meshes/environment/ZenPoolWithToolBoxCollision.stl"/>
         </geometry>
         <origin rpy="0 0 0" xyz="0.0 0.0 0.0"/>
@@ -55,5 +55,5 @@
       <visual>
         <geometry>
-          <mesh filename="package://my_robot_cell_description/meshes/ToolBoxPlatform.stl" />
+          <mesh filename="package://my_robot_cell_description/meshes/environment/ToolBoxPlatform.stl" />
         </geometry>
         <origin rpy="0 0 ${pi}" xyz="${0.25 - 0.045/2} 0 ${0.195/2}"/>
@@ -62,5 +62,5 @@
       <collision>
         <geometry>
-          <mesh filename="package://my_robot_cell_description/meshes/ToolBoxPlatform.stl" />
+          <mesh filename="package://my_robot_cell_description/meshes/environment/ToolBoxPlatform.stl" />
         </geometry>
         <origin rpy="0 0 ${pi}" xyz="${0.25 - 0.045/2} 0 ${0.195/2}"/>
@@ -75,5 +75,5 @@
       <visual>
         <geometry>
-          <mesh filename="package://my_robot_cell_description/meshes/ToolBoxes.stl" />
+          <mesh filename="package://my_robot_cell_description/meshes/environment/ToolBoxes.stl" />
         </geometry>
         <origin rpy="0 0 ${pi}" xyz="${0.25 - 0.045/2} 0 ${0.195/2}"/>
@@ -82,5 +82,5 @@
       <collision>
         <geometry>
-          <mesh filename="package://my_robot_cell_description/meshes/ToolBoxes.stl" />
+          <mesh filename="package://my_robot_cell_description/meshes/environment/ToolBoxes.stl" />
         </geometry>
         <origin rpy="0 0 ${pi}" xyz="${0.25 - 0.045/2} 0 ${0.195/2}"/>
@@ -108,5 +108,5 @@
       <visual>
         <geometry>
-          <mesh filename="package://my_robot_cell_description/meshes/ToolChangerArmSide.stl"/>
+          <mesh filename="package://my_robot_cell_description/meshes/tool_changer/ToolChangerArmSide.stl"/>
         </geometry>
         <origin rpy="${pi} 0 0" xyz="0 0.0 -0.0248"/>
@@ -115,5 +115,5 @@
       <collision>
         <geometry>
-          <mesh filename="package://my_robot_cell_description/meshes/ToolChangerArmSide.stl"/>
+          <mesh filename="package://my_robot_cell_description/meshes/tool_changer/ToolChangerArmSide.stl"/>
         </geometry>
         <origin rpy="${pi} 0 0" xyz="0 0.0 -0.0248"/>
@@ -128,5 +128,5 @@
       <visual>
         <geometry>
-          <mesh filename="package://my_robot_cell_description/meshes/CleanerTool.stl" scale="0.001 0.001 0.001"/>
+          <mesh filename="package://my_robot_cell_description/meshes/end_effectors/CleanerTool.stl" scale="0.001 0.001 0.001"/>
         </geometry>
         <origin rpy="0 ${pi} 0" xyz="-0.031739 0.039119 -0.097"/>
@@ -135,5 +135,5 @@
       <collision>
         <geometry>
-          <mesh filename="package://my_robot_cell_description/meshes/CleanerTool.stl" scale="0.001 0.001 0.001"/>
+          <mesh filename="package://my_robot_cell_description/meshes/end_effectors/CleanerTool.stl" scale="0.001 0.001 0.001"/>
         </geometry>
         <origin rpy="0 ${pi} 0" xyz="-0.031739 0.039119 -0.097"/>
@@ -148,5 +148,5 @@
       <visual>
         <geometry>
-          <mesh filename="package://my_robot_cell_description/meshes/PenTool.stl" scale="0.001 0.001 0.001"/>
+          <mesh filename="package://my_robot_cell_description/meshes/end_effectors/PenTool.stl" scale="0.001 0.001 0.001"/>
         </geometry>
         <origin rpy="0 ${pi} 0" xyz="-0.016839 0.039119 -0.097"/>
@@ -155,5 +155,5 @@
       <collision>
         <geometry>
-          <mesh filename="package://my_robot_cell_description/meshes/PenTool.stl" scale="0.001 0.001 0.001"/>
+          <mesh filename="package://my_robot_cell_description/meshes/end_effectors/PenTool.stl" scale="0.001 0.001 0.001"/>
         </geometry>
         <origin rpy="0 ${pi} 0" xyz="-0.016839 0.039119 -0.097"/>

Commit message: last two 1 day

File: my_robot_cell/my_robot_cell_description/urdf/my_robot_cell_macro.xacro (robot description, xacro)
@@ -46,4 +46,11 @@
       </collision>
     </link>
+    <!-- Dummy frame rotated 180 degrees so +X points exactly where the user wants -->
+    <link name="pool_actual"/>
+    <joint name="pool_to_pool_actual" type="fixed">
+      <parent link="pool"/>
+      <child link="pool_actual"/>
+      <origin xyz="0 0 0" rpy="0 0 ${pi}" />
+    </joint>
     <link name="robot_mount"/>
     <joint name="base_to_robot_mount" type="fixed">
@@ -52,44 +59,4 @@
       <origin xyz="0.0 0.0 0" rpy="0 0 ${- 5*pi/4}" />
     </joint>
-    <!-- <link name="tool_box">
-      <visual>
-        <geometry>
-          <mesh filename="package://my_robot_cell_description/meshes/environment/ToolBoxPlatform.stl" />
-        </geometry>
-        <origin rpy="0 0 ${pi}" xyz="${0.25 - 0.045/2} 0 ${0.195/2}"/>
-        <material name="white" />
-      </visual>
-      <collision>
-        <geometry>
-          <mesh filename="package://my_robot_cell_description/meshes/environment/ToolBoxPlatform.stl" />
-        </geometry>
-        <origin rpy="0 0 ${pi}" xyz="${0.25 - 0.045/2} 0 ${0.195/2}"/>
-      </collision>
-    </link>
-    <joint name="pool_toolbox_platform_joint" type="fixed">
-      <parent link="pool" />
-      <child link="tool_box" />
-      <origin xyz="-.2275 .0 -.115" rpy="0 0 0" />
-    </joint>
-    <link name="tools">
-      <visual>
-        <geometry>
-          <mesh filename="package://my_robot_cell_description/meshes/environment/ToolBoxes.stl" />
-        </geometry>
-        <origin rpy="0 0 ${pi}" xyz="${0.25 - 0.045/2} 0 ${0.195/2}"/>
-        <material name="red" />
-      </visual>
-      <collision>
-        <geometry>
-          <mesh filename="package://my_robot_cell_description/meshes/environment/ToolBoxes.stl" />
-        </geometry>
-        <origin rpy="0 0 ${pi}" xyz="${0.25 - 0.045/2} 0 ${0.195/2}"/>
-      </collision>
-    </link>
-    <joint name="pool_toolboxes_joint" type="fixed">
-      <parent link="pool" />
-      <child link="tools" />
-      <origin xyz="-.2275 .0 -.115" rpy="0 0 0" />
-    </joint> -->
     <!--This will create the specific robot-->
     <xacro:ur_robot
@@ -125,44 +92,4 @@
       <origin rpy="0 0 0" xyz="0.0 0.0 0.02"/>
     </joint>
-    <!-- <link name="cleaner_tool">
-      <visual>
-        <geometry>
-          <mesh filename="package://my_robot_cell_description/meshes/end_effectors/CleanerTool.stl" scale="0.001 0.001 0.001"/>
-        </geometry>
-        <origin rpy="0 ${pi} 0" xyz="-0.031739 0.039119 -0.097"/>
-        <material name="blue"/>
-      </visual>
-      <collision>
-        <geometry>
-          <mesh filename="package://my_robot_cell_description/meshes/end_effectors/CleanerTool.stl" scale="0.001 0.001 0.001"/>
-        </geometry>
-        <origin rpy="0 ${pi} 0" xyz="-0.031739 0.039119 -0.097"/>
-      </collision>
-    </link>
-    <joint name="cleaner_to_tc" type="fixed">
-      <parent link="tc_arm_side"/>
-      <child link="cleaner_tool" />
-      <origin rpy="0 0 0" xyz="0.0 0.0 ${0.115}"/>
-    </joint>
-    <link name="pen_tool">
-      <visual>
-        <geometry>
-          <mesh filename="package://my_robot_cell_description/meshes/end_effectors/PenTool.stl" scale="0.001 0.001 0.001"/>
-        </geometry>
-        <origin rpy="0 ${pi} 0" xyz="-0.016839 0.039119 -0.097"/>
-        <material name="green"/>
-      </visual>
-      <collision>
-        <geometry>
-          <mesh filename="package://my_robot_cell_description/meshes/end_effectors/PenTool.stl" scale="0.001 0.001 0.001"/>
-        </geometry>
-        <origin rpy="0 ${pi} 0" xyz="-0.016839 0.039119 -0.097"/>
-      </collision>
-    </link>
-    <joint name="pen_to_tc" type="fixed">
-      <parent link="tc_arm_side"/>
-      <child link="pen_tool" />
-      <origin rpy="0 0 0" xyz="0.0 0.0 ${0.115}"/>
-    </joint> -->
   </xacro:macro>
 </robot>
